Commit message: update

File: legged_lab/assets/elf3_lite/urdf/elf3.urdf (robot description, URDF)
Before this commit: robot elf3, 30 links, 29 joints
Links:
- added link d435i_link
- added link head_y_link, mass 1.57425673; collision mesh filename=./meshes/head_y_link.STL; visual mesh filename=./meshes/head_y_link.STL
- added link head_z_link, mass 0.37665142; collision mesh filename=./meshes/head_z_link.STL; visual mesh filename=./meshes/head_z_link.STL
- added link imu_link
- added link mid360_link
- added link torso_front_bottom_d435i_link
- link l_ankle_x_link: mass 0.298065216713201 -> 0.37980156; geometry collision mesh filename=./meshes/l_ankle_x_link.STL; visual mesh filename=./meshes/l_ankle_x_link.STL
- link l_ankle_y_link: mass 0.0126898593121342 -> 0.01268984; geometry visual mesh filename=./meshes/l_ankle_y_link.STL
- link l_elbow_y_link: mass 0.0938669247468512 -> 0.1020615; geometry visual mesh filename=./meshes/l_elbow_y_link.STL
- link l_hip_x_link: mass 0.214152254706427 -> 0.23202193; geometry visual mesh filename=./meshes/l_hip_x_link.STL
- link l_hip_y_link: mass 1.70384733340318 -> 1.74663835; geometry collision mesh filename=./meshes/l_hip_y_link.STL; visual mesh filename=./meshes/l_hip_y_link.STL
- link l_hip_z_link: mass 2.84278184760334 -> 2.94332059; geometry collision mesh filename=./meshes/l_hip_z_link.STL; visual mesh filename=./meshes/l_hip_z_link.STL
- link l_knee_y_link: mass 1.77390809 -> 1.86991215; geometry visual mesh filename=./meshes/l_knee_y_link.STL
- link l_shoulder_x_link: mass 0.130650985436178 -> 0.13939414; geometry visual mesh filename=./meshes/l_shoulder_x_link.STL
- link l_shoulder_y_link: mass 0.938482977144261 -> 0.99747353; geometry visual mesh filename=./meshes/l_shoulder_y_link.STL
- link l_shoulder_z_link: mass 1.29694131347632 -> 1.67349896; geometry collision mesh filename=./meshes/l_shoulder_z_link.STL; visual mesh filename=./meshes/l_shoulder_z_link.STL
- link l_wrist_x_link: mass 0.65867493591403 -> 1.24945755; geometry collision mesh filename=./meshes/l_wrist_x_link_part.STL; visual mesh filename=./meshes/l_wrist_x_link.STL
- link l_wrist_y_link: mass 0.243805170394381 -> 0.56828784; geometry collision mesh filename=./meshes/l_wrist_y_link.STL; visual mesh filename=./meshes/l_wrist_y_link.STL
- link l_wrist_z_link: mass 0.106560860250811 -> 0.09977741; geometry collision mesh filename=./meshes/l_wrist_z_link.STL; visual mesh filename=./meshes/l_wrist_z_link.STL
- link r_ankle_x_link: mass 0.298065216713202 -> 0.37980156; geometry collision mesh filename=./meshes/r_ankle_x_link.STL; visual mesh filename=./meshes/r_ankle_x_link.STL
- link r_ankle_y_link: mass 0.0126898593121342 -> 0.01268984; geometry visual mesh filename=./meshes/r_ankle_y_link.STL
- link r_elbow_y_link: mass 0.0938669107317605 -> 0.1020615; geometry visual mesh filename=./meshes/r_elbow_y_link.STL
- link r_hip_x_link: mass 0.214152254706428 -> 0.23202193; geometry visual mesh filename=./meshes/r_hip_x_link.STL
- link r_hip_y_link: mass 1.70384734270319 -> 1.74663841; geometry collision mesh filename=./meshes/r_hip_y_link.STL; visual mesh filename=./meshes/r_hip_y_link.STL
- link r_hip_z_link: mass 2.8427830619077 -> 2.94332069; geometry collision mesh filename=./meshes/r_hip_z_link.STL; visual mesh filename=./meshes/r_hip_z_link.STL
- link r_knee_y_link: mass 1.77390996 -> 1.86991402; geometry visual mesh filename=./meshes/r_knee_y_link.STL
- link r_shoulder_x_link: mass 0.130650985436178 -> 0.13939414; geometry visual mesh filename=./meshes/r_shoulder_x_link.STL
- link r_shoulder_y_link: mass 0.938482977205647 -> 0.99747344; geometry visual mesh filename=./meshes/r_shoulder_y_link.STL
- link r_shoulder_z_link: mass 1.29694127388881 -> 1.67349843; geometry collision mesh filename=./meshes/r_shoulder_z_link.STL; visual mesh filename=./meshes/r_shoulder_z_link.STL
- link r_wrist_x_link: mass 0.658674935909524 -> 1.24945755; geometry collision mesh filename=./meshes/r_wrist_x_link_part.STL; visual mesh filename=./meshes/r_wrist_x_link.STL
- link r_wrist_y_link: mass 0.243805170389875 -> 0.56828784; geometry collision mesh filename=./meshes/r_wrist_y_link.STL; visual mesh filename=./meshes/r_wrist_y_link.STL
- link r_wrist_z_link: mass 0.106560859874613 -> 0.09977741; geometry collision mesh filename=./meshes/r_wrist_z_link.STL; visual mesh filename=./meshes/r_wrist_z_link.STL
- link torso_link: mass 12.004 -> 11.66386158; geometry collision mesh filename=./meshes/torso_link.STL; visual mesh filename=./meshes/torso_link.STL
- link waist_x_link: mass 0.215642587680923 -> 0.24344947; geometry visual mesh filename=./meshes/waist_x_link.STL
- link waist_y_link: mass 0.0661517869264427 -> 0.06620328; geometry visual mesh filename=./meshes/waist_y_link.STL
- link waist_z_link: mass 4.95603362274037 -> 5.2693813; geometry visual mesh filename=./meshes/waist_z_link.STL
Joints:
- added joint d435i_joint: type fixed, parent head_y_link, child d435i_link, origin xyz=0.0628 0.0175 -0.048 rpy=-1.5708 0 -1.5708, axis 0 0 0
- added joint head_y_joint: type revolute, parent head_z_link, child head_y_link, origin xyz=0 0 0 rpy=0 0 0, axis 0 1 0, limit lower=-0.785 upper=0.785 effort=21 velocity=20
- added joint head_z_joint: type revolute, parent torso_link, child head_z_link, origin xyz=0 0 0.2995 rpy=0 0 0, axis 0 0 1, limit lower=-1.57 upper=1.57 effort=21 velocity=20
- added joint imu_joint: type fixed, parent torso_link, child imu_link, origin xyz=0 0 0 rpy=0 0 0, axis 0 0 0
- added joint mid360_joint: type fixed, parent head_y_link, child mid360_link, origin xyz=0 0 -0.081 rpy=3.1416 0 0, axis 0 0 0
- added joint torso_front_bottom_d435i_joint: type fixed, parent torso_link, child torso_front_bottom_d435i_link, origin xyz=0.1152 0.0175 -0.1358 rpy=-2.7925 0 -1.5708, axis 0 0 0
- joint l_ankle_x_joint: limit lower=-0.34907 upper=0.34907 effort=50 velocity=20 -> lower=-0.34907 upper=0.34907 effort=20 velocity=20
- joint l_elbow_y_joint: limit lower=-0.95993 upper=1.6581 effort=50 velocity=20 -> lower=-0.95993 upper=1.6581 effort=45 velocity=20
- joint l_hip_x_joint: limit lower=-0.48869 upper=3.0543 effort=100 velocity=20 -> lower=-0.48869 upper=3.0543 effort=150 velocity=20
- joint l_hip_y_joint: limit lower=-2.8798 upper=2.8798 effort=100 velocity=20 -> lower=-2.8798 upper=2.8798 effort=150 velocity=20
- joint l_hip_z_joint: limit lower=-2.8798 upper=2.8798 effort=50 velocity=20 -> lower=-2.8798 upper=2.8798 effort=45 velocity=20
- joint l_shoulder_x_joint: limit lower=-0.34907 upper=3.0543 effort=50 velocity=20 -> lower=-0.34907 upper=3.0543 effort=45 velocity=20
- joint l_shoulder_y_joint: limit lower=-2.8798 upper=2.8798 effort=50 velocity=20 -> lower=-2.8798 upper=2.8798 effort=45 velocity=20
- joint l_shoulder_z_joint: limit lower=-2.8798 upper=2.8798 effort=25 velocity=20 -> lower=-2.8798 upper=2.8798 effort=21 velocity=20
- joint l_wrist_x_joint: limit lower=-2.8798 upper=2.8798 effort=25 velocity=20 -> lower=-2.8798 upper=2.8798 effort=21 velocity=20
- joint l_wrist_y_joint: limit lower=-1.309 upper=1.309 effort=25 velocity=20 -> lower=-1.309 upper=1.309 effort=21 velocity=20
- joint l_wrist_z_joint: limit lower=-0.7854 upper=0.7854 effort=25 velocity=20 -> lower=-0.7854 upper=0.7854 effort=21 velocity=20
- joint r_ankle_x_joint: limit lower=-0.34907 upper=0.34907 effort=50 velocity=20 -> lower=-0.34907 upper=0.34907 effort=20 velocity=20
- joint r_elbow_y_joint: limit lower=-0.95993 upper=1.6581 effort=50 velocity=20 -> lower=-0.95993 upper=1.6581 effort=45 velocity=20
- joint r_hip_x_joint: limit lower=-3.0543 upper=0.48869 effort=100 velocity=20 -> lower=-3.0543 upper=0.48869 effort=150 velocity=20
- joint r_hip_y_joint: limit lower=-2.8798 upper=2.8798 effort=100 velocity=20 -> lower=-2.8798 upper=2.8798 effort=150 velocity=20
- joint r_hip_z_joint: limit lower=-2.8798 upper=2.8798 effort=50 velocity=20 -> lower=-2.8798 upper=2.8798 effort=45 velocity=20
- joint r_shoulder_x_joint: limit lower=-3.0543 upper=0.34907 effort=50 velocity=20 -> lower=-3.0543 upper=0.34907 effort=45 velocity=20
- joint r_shoulder_y_joint: limit lower=-2.8798 upper=2.8798 effort=50 velocity=20 -> lower=-2.8798 upper=2.8798 effort=45 velocity=20
- joint r_shoulder_z_joint: limit lower=-2.8798 upper=2.8798 effort=25 velocity=20 -> lower=-2.8798 upper=2.8798 effort=21 velocity=20
- joint r_wrist_x_joint: limit lower=-2.8798 upper=2.8798 effort=25 velocity=20 -> lower=-2.8798 upper=2.8798 effort=21 velocity=20
- joint r_wrist_y_joint: limit lower=-1.309 upper=1.309 effort=25 velocity=20 -> lower=-1.309 upper=1.309 effort=21 velocity=20
- joint r_wrist_z_joint: limit lower=-0.7854 upper=0.7854 effort=25 velocity=20 -> lower=-0.7854 upper=0.7854 effort=21 velocity=20
- joint waist_y_joint: limit lower=-0.5236 upper=0.5236 effort=100 velocity=20 -> lower=-0.5236 upper=0.5236 effort=90 velocity=20
- joint waist_z_joint: limit lower=-2.8798 upper=2.8798 effort=100 velocity=20 -> lower=-2.8798 upper=2.8798 effort=150 velocity=20
